File: hardware/Eagle Files/Open_IR_Blaster.sch (EAGLE design)
At the start: 36 parts, among them J1 4907, Q1 IRLML6344TRPBF, U1 AZ1117EH-1.5TRG1

Commit message: Adds indicator LED to board and pulldown for MOSFET (not required).
Parts:
- removed H1: MOUNT-HOLE3.2, holes:MOUNT-HOLE3.2
- added LED9: (no value), adafruit:LEDCHIP-LED0603
- added R18: 4.7k, adafruit:R-US_R0603
- added R19: 100k, adafruit:R-US_R0603
Connections:
- new net N$13: LED9.C, R18.2
- net +5VDC: now also LED9.A
- net GND: now also R19.1
- net N$12: now also R19.2
- net N$9: now also R18.1
